File: pcb_design/motor_board/Motorboard.brd (EAGLE design)
At the start: 31 x 31 mm, 75 parts, among them M1 STEPPER_MOTOR_SMD, M2 STEPPER_MOTOR_SMD

Commit message: Minor silk screen changes to mMotor board
Parts:
- ATMEGA328P: value ATMEGA168 -> ATMEGA328
- JP_CHRG_L, JP_CHRG_R: value M01NOSILK-KIT -> (none)
- renumbered ATMEGA168P to ATMEGA328P
Connections:
- net VBAT renamed VDD
Changed lines of the file:
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@@
 <attribute name="NAME" x="20.6" y="23.662" size="0.6096" layer="22" font="vector" rot="MR0"/>
 </element>
-<element name="ATMEGA168P" library="GRITSBot" package="TQFP32-08" value="ATMEGA168" x="15.5" y="17" smashed="yes" rot="MR0"/>
+<element name="ATMEGA328P" library="GRITSBot" package="TQFP32-08" value="ATMEGA328" x="15.5" y="17" smashed="yes" rot="MR0"/>
 <element name="LED_RIGHT" library="SparkFun-LED" package="LED-0603" value="green" x="27.2" y="23.2" smashed="yes" rot="MR90"/>
 <element name="R1" library="SparkFun-Resistors" package="0603" value="1k" x="29.7" y="25.8" smashed="yes" rot="MR270">
@@
 </element>
 <element name="JP5" library="abes" package="FIDUCIAL-1X2.5" value="FIDUCIAL1X2.5" x="5" y="3.5" smashed="yes" rot="MR0"/>
-<element name="JP_CHRG_L" library="SparkFun-Connectors" package="1X01NS-KIT" value="M01NOSILK-KIT" x="7.5" y="1.5"/>
-<element name="JP_CHRG_R" library="SparkFun-Connectors" package="1X01NS-KIT" value="M01NOSILK-KIT" x="23.5" y="1.5"/>
+<element name="JP_CHRG_L" library="SparkFun-Connectors" package="1X01NS-KIT" value="" x="7.5" y="1.5"/>
+<element name="JP_CHRG_R" library="SparkFun-Connectors" package="1X01NS-KIT" value="" x="23.5" y="1.5"/>
 <element name="CUR_RIGHT" library="GRITSBot" package="SOT23-3" value="ZXCT1009_CURRENT" x="17.2" y="4.9" smashed="yes" rot="MR270">
 <attribute name="VALUE" x="17.3905" y="5.916" size="0.4064" layer="28" rot="MR270"/>
@@
 <vertex x="31" y="31"/>
 </polygon>
-<contactref element="ATMEGA168P" pad="5"/>
-<contactref element="ATMEGA168P" pad="3"/>
-<contactref element="ATMEGA168P" pad="21"/>
+<contactref element="ATMEGA328P" pad="5"/>
+<contactref element="ATMEGA328P" pad="3"/>
+<contactref element="ATMEGA328P" pad="21"/>
 <contactref element="R1" pad="1"/>
 <contactref element="LINE_SENSE_2" pad="4"/>
@@
 <contactref element="R6" pad="2"/>
 <contactref element="R8" pad="2"/>
-<contactref element="ATMEGA168P" pad="18"/>
-<contactref element="ATMEGA168P" pad="4"/>
-<contactref element="ATMEGA168P" pad="6"/>
-<contactref element="ATMEGA168P" pad="20"/>
+<contactref element="ATMEGA328P" pad="18"/>
+<contactref element="ATMEGA328P" pad="4"/>
+<contactref element="ATMEGA328P" pad="6"/>
+<contactref element="ATMEGA328P" pad="20"/>
 <contactref element="R2" pad="2"/>
 <wire x1="14.2" y1="16.6" x2="11.2074" y2="16.6" width="0.254" layer="16"/>
@@
 </signal>
 <signal name="M2IN3">
-<contactref element="ATMEGA168P" pad="8"/>
+<contactref element="ATMEGA328P" pad="8"/>
 <contactref element="MOTOR_CTRL_R" pad="13"/>
 <via x="23.8" y="13.9" extent="1-16" drill="0.381"/>
@@
 </signal>
 <signal name="M2IN4">
-<contactref element="ATMEGA168P" pad="7"/>
+<contactref element="ATMEGA328P" pad="7"/>
 <contactref element="MOTOR_CTRL_R" pad="9"/>
 <via x="22.6" y="15" extent="1-16" drill="0.381"/>
@@
 </signal>
 <signal name="M2IN1">
-<contactref element="ATMEGA168P" pad="9"/>
+<contactref element="ATMEGA328P" pad="9"/>
 <contactref element="MOTOR_CTRL_R" pad="2"/>
 <via x="19.2926" y="11.9074" extent="1-16" drill="0.381"/>
@@
 </signal>
 <signal name="M2IN2">
-<contactref element="ATMEGA168P" pad="10"/>
+<contactref element="ATMEGA328P" pad="10"/>
 <contactref element="MOTOR_CTRL_R" pad="6"/>
 <wire x1="18.7" y1="10.8" x2="17.5" y2="12" width="0.254" layer="16"/>
@@
 </signal>
 <signal name="M1IN1">
-<contactref element="ATMEGA168P" pad="13"/>
+<contactref element="ATMEGA328P" pad="13"/>
 <contactref element="MOTOR_CTRL_L" pad="2"/>
 <wire x1="15.1" y1="12.7074" x2="15.1" y2="11.1" width="0.254" layer="16"/>
@@
 </signal>
 <signal name="M1IN2">
-<contactref element="ATMEGA168P" pad="14"/>
+<contactref element="ATMEGA328P" pad="14"/>
 <contactref element="MOTOR_CTRL_L" pad="6"/>
 <via x="5.9" y="6.6" extent="1-16" drill="0.381"/>
@@
 </signal>
 <signal name="M1IN3">
-<contactref element="ATMEGA168P" pad="12"/>
+<contactref element="ATMEGA328P" pad="12"/>
 <contactref element="MOTOR_CTRL_L" pad="13"/>
 <via x="4.5" y="10.4" extent="1-16" drill="0.381"/>
@@
 </signal>
 <signal name="M1IN4">
-<contactref element="ATMEGA168P" pad="11"/>
+<contactref element="ATMEGA328P" pad="11"/>
 <contactref element="MOTOR_CTRL_L" pad="9"/>
 <wire x1="16.7" y1="12.7074" x2="16.7" y2="11.1" width="0.254" layer="16"/>
@@
 </signal>
 <signal name="MOSI">
-<contactref element="ATMEGA168P" pad="15"/>
+<contactref element="ATMEGA328P" pad="15"/>
 <via x="17.1" y="14" extent="1-16" drill="0.381"/>
 <wire x1="17.1" y1="14" x2="13.9" y2="14" width="0.254" layer="16"/>
@@
 </signal>
 <signal name="MISO">
-<contactref element="ATMEGA168P" pad="16"/>
+<contactref element="ATMEGA328P" pad="16"/>
 <wire x1="17.1" y1="24.5" x2="17.1" y2="15.4" width="0.254" layer="1"/>
 <via x="16.4" y="14.7" extent="1-16" drill="0.381"/>
@@
 </signal>
 <signal name="SCK">
-<contactref element="ATMEGA168P" pad="17"/>
+<contactref element="ATMEGA328P" pad="17"/>
 <wire x1="16.6" y1="23.9" x2="16.6" y2="15.9" width="0.254" layer="1"/>
 <wire x1="11.2074" y1="14.2" x2="12.1" y2="14.2" width="0.254" layer="16"/>
@@
 </signal>
 <signal name="RESET">
-<contactref element="ATMEGA168P" pad="29"/>
+<contactref element="ATMEGA328P" pad="29"/>
 <contactref element="R2" pad="1"/>
 <via x="15.9" y="20" extent="1-16" drill="0.381"/>
@@
 <signal name="LINE_RIGHT">
 <contactref element="R7" pad="2"/>
-<contactref element="ATMEGA168P" pad="31"/>
+<contactref element="ATMEGA328P" pad="31"/>
 <wire x1="22.7" y1="22.3" x2="17.8" y2="22.3" width="0.254" layer="16"/>
 <wire x1="17.8" y1="22.3" x2="17.5" y2="22" width="0.254" layer="16"/>
@@
 <wire x1="3.9" y1="23.9" x2="3.5" y2="24.3" width="0.254" layer="16"/>
 <wire x1="3.5" y1="24.3" x2="3.5" y2="24.95" width="0.254" layer="16"/>
-<contactref element="ATMEGA168P" pad="30"/>
+<contactref element="ATMEGA328P" pad="30"/>
 <wire x1="16.7" y1="21.2926" x2="16.7" y2="19.6" width="0.254" layer="16"/>
 <wire x1="16.7" y1="19.6" x2="16.4" y2="19.3" width="0.254" layer="16"/>
@@
 <wire x1="27.55" y1="24.9" x2="27.6" y2="24.95" width="0.254" layer="16"/>
 </signal>
-<signal name="VBAT">
+<signal name="VDD">
 <contactref element="JP_POWER" pad="2"/>
 <wire x1="19.65" y1="3.35" x2="19.3" y2="3" width="0.3048" layer="16"/>
@@
 </signal>
 <signal name="A4_SDA">
-<contactref element="ATMEGA168P" pad="27"/>
+<contactref element="ATMEGA328P" pad="27"/>
 <contactref element="JP_I2C" pad="2"/>
 <wire x1="14.3" y1="21.2926" x2="14.3" y2="22.8" width="0.254" layer="16"/>
@@
 </signal>
 <signal name="A5_SCL">
-<contactref element="ATMEGA168P" pad="28"/>
+<contactref element="ATMEGA328P" pad="28"/>
 <contactref element="JP_I2C" pad="1"/>
 <wire x1="15.1" y1="21.2926" x2="15.1" y2="22.5" width="0.254" layer="16"/>
@@
 </signal>
 <signal name="AD3_LINE_RIGHT">
-<contactref element="ATMEGA168P" pad="26"/>
+<contactref element="ATMEGA328P" pad="26"/>
 <contactref element="R8" pad="1"/>
 <contactref element="LINE_SENSE_1" pad="1"/>
@@
 </signal>
 <signal name="AD2_LINE_LEFT">
-<contactref element="ATMEGA168P" pad="25"/>
+<contactref element="ATMEGA328P" pad="25"/>
 <contactref element="R6" pad="1"/>
 <contactref element="LINE_SENSE_2" pad="1"/>
@@
 <signal name="LED_LEFT">
 <contactref element="LED_LEFT" pad="A"/>
-<contactref element="ATMEGA168P" pad="32"/>
+<contactref element="ATMEGA328P" pad="32"/>
 <via x="14.5" y="19.1" extent="1-16" drill="0.381"/>
 <wire x1="14.5" y1="19.1" x2="14.2" y2="19.1" width="0.254" layer="1"/>
@@
 <signal name="LED_RIGHT">
 <contactref element="LED_RIGHT" pad="A"/>
-<contactref element="ATMEGA168P" pad="2"/>
+<contactref element="ATMEGA328P" pad="2"/>
 <wire x1="21.1" y1="21.8" x2="20.8" y2="21.5" width="0.254" layer="16"/>
 <wire x1="20.8" y1="21.5" x2="20.8" y2="19.3" width="0.254" layer="16"/>
@@
 <signal name="TEMP_LEFT">
 <contactref element="TEMP_LEFT" pad="1"/>
-<contactref element="ATMEGA168P" pad="22"/>
+<contactref element="ATMEGA328P" pad="22"/>
 <wire x1="11.2074" y1="18.2" x2="9.6" y2="18.2" width="0.254" layer="16"/>
 <wire x1="9.6" y1="18.2" x2="7.65" y2="20.15" width="0.254" layer="16"/>
@@
 <signal name="TEMP_RIGHT">
 <contactref element="TEMP_RIGHT" pad="1"/>
-<contactref element="ATMEGA168P" pad="19"/>
+<contactref element="ATMEGA328P" pad="19"/>
 <wire x1="23.7" y1="20.6" x2="22" y2="20.6" width="0.254" layer="16"/>
 <wire x1="22" y1="20.6" x2="21.8" y2="20.4" width="0.254" layer="16"/>
@@
 <wire x1="16.35" y1="8.15" x2="16" y2="8.5" width="0.254" layer="16"/>
 <wire x1="13.7" y1="9" x2="13.4" y2="9.3" width="0.254" layer="16"/>
-<contactref element="ATMEGA168P" pad="24"/>
+<contactref element="ATMEGA328P" pad="24"/>
 <wire x1="13.4" y1="9.3" x2="13.4" y2="11.5" width="0.254" layer="16"/>
 <via x="13.4" y="11.5" extent="1-16" drill="0.381"/>
@@
 <contactref element="R10" pad="2"/>
 <contactref element="CUR_LEFT" pad="3"/>
-<contactref element="ATMEGA168P" pad="23"/>
+<contactref element="ATMEGA328P" pad="23"/>
 <via x="12.5" y="11.5" extent="1-16" drill="0.381"/>
 <wire x1="12.5" y1="11.5" x2="12.5" y2="17.4" width="0.254" layer="1"/>
@@
 </signal>
 <signal name="ESP_RESET">
-<contactref element="ATMEGA168P" pad="1"/>
+<contactref element="ATMEGA328P" pad="1"/>
 <contactref element="JP_RST" pad="2"/>
 <wire x1="19.7926" y1="19.8" x2="18.3" y2="19.8" width="0.254" layer="16"/>
